File: hardware/temperature-humidity-controller-tryout.sch (KiCad schematic (older format))
At the start: 0 parts

Commit message: update,
Changed lines of the file:
@@
 EESchema Schematic File Version 4
+LIBS:temperature-humidity-controller-tryout-cache
 EELAYER 29 0
 EELAYER END
 $Descr User 8500 5500
 encoding utf-8
-Sheet 1 1
+Sheet 1 9
 Title ""
 Date ""
@@
 Text Notes 3950 4250 0    50   ~ 0
 temperature\nhumidity\nrelay control\n\nhko connect
+$Sheet
+S 3400 1300 1200 1650
+U 5D1EF826
+F0 "ESP-12" 50
+F1 "ESP-12.sch" 50
+$EndSheet
+$Sheet
+S 600  4000 800  700
+U 5D1F27E8
+F0 "power" 50
+F1 "power.sch" 50
+$EndSheet
+$Sheet
+S 1500 1300 800  700
+U 5D1F280A
+F0 "sensor" 50
+F1 "sensor.sch" 50
+$EndSheet
+$Sheet
+S 5600 1350 750  600
+U 5D1F3E01
+F0 "relay1" 50
+F1 "relay1.sch" 50
+$EndSheet
+$Sheet
+S 5600 2250 750  600
+U 5D1F3E80
+F0 "relay2" 50
+F1 "relay2.sch" 50
+$EndSheet
+$Sheet
+S 1500 2250 800  700
+U 5D1F7924
+F0 "ssd1306" 50
+F1 "ssd1306.sch" 50
+$EndSheet
 $EndSCHEMATC
